File: mcp1642b.sch (EAGLE design)
At the start: 6 parts, among them U11 MCP1642B

Commit message: Mon 28 Jan 2019 22:16:21 EST - updated MCP1642 device with planes
Connections:
- net N$1 renamed SW
Changed lines of the file:
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@@
 </segment>
 </net>
-<net name="N$1" class="0">
+<net name="SW" class="0">
 <segment>
 <pinref part="U11" gate="G$1" pin="SW"/>
 <pinref part="L1" gate="G$1" pin="1"/>
 <wire x1="38.1" y1="35.56" x2="38.1" y2="33.02" width="0.1524" layer="91"/>
+<label x="40.64" y="35.56" size="1.016" layer="95" xref="yes"/>
 </segment>
 </net>
