File: mcp1642b.brd (EAGLE design)
At the start: 16 x 35 mm, 6 parts, among them U11 MCP1642B

Commit message: Wed  6 Mar 2019 10:52:50 EST - added AAA alkaline version of TPS61032
Parts:
- C1, C2: value 10uF -> 47uF
Changed lines of the file:
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@@
 <?xml version="1.0" encoding="utf-8"?>
 <!DOCTYPE eagle SYSTEM "eagle.dtd">
-<eagle version="9.0.1">
+<eagle version="9.0.0">
 <drawing>
 <settings>
@@
 <layer number="220" name="220bmp" color="21" fill="1" visible="no" active="no"/>
 <layer number="221" name="221bmp" color="22" fill="1" visible="no" active="no"/>
+<layer number="222" name="222bmp" color="23" fill="1" visible="no" active="no"/>
 <layer number="223" name="223bmp" color="24" fill="1" visible="no" active="no"/>
 <layer number="224" name="224bmp" color="25" fill="1" visible="no" active="no"/>
@@
 </autorouter>
 <elements>
-<element name="C1" library="rcl" package="153CLV-0505" value="10uF" x="11.25" y="14" rot="R180"/>
-<element name="C2" library="rcl" package="153CLV-0505" value="10uF" x="11.25" y="25.5"/>
+<element name="C1" library="rcl" library_urn="urn:adsk.eagle:library:334" package="153CLV-0505" package3d_urn="urn:adsk.eagle:package:23402/1" value="47uF" x="11.25" y="14" rot="R180">
+<attribute name="SPICEPREFIX" value="C" x="11.25" y="14" size="1.778" layer="27" rot="R180" display="off"/>
+</element>
+<element name="C2" library="rcl" library_urn="urn:adsk.eagle:library:334" package="153CLV-0505" package3d_urn="urn:adsk.eagle:package:23402/1" value="47uF" x="11.25" y="25.5">
+<attribute name="SPICEPREFIX" value="C" x="11.25" y="25.5" size="1.778" layer="27" display="off"/>
+</element>
 <element name="J1" library="SparkFun-Connectors" library_urn="urn:adsk.eagle:library:513" package="JST-2-SMD" package3d_urn="urn:adsk.eagle:package:38042/1" value="" x="8" y="4" rot="R180">
 <attribute name="PROD_ID" value="CONN-11443" x="8" y="4" size="1.778" layer="27" rot="R180" display="off"/>
@@
 </element>
 <element name="J2" library="SparkFun-Connectors" library_urn="urn:adsk.eagle:library:513" package="1X02_XTRA_BIG" package3d_urn="urn:adsk.eagle:package:38054/1" value="" x="8.144" y="32.258" rot="R180"/>
-<element name="L1" library="rcl" package="POWER-CHOKE_WE-TPC" value="4.7uH" x="4.25" y="19"/>
+<element name="L1" library="rcl" library_urn="urn:adsk.eagle:library:334" package="POWER-CHOKE_WE-TPC" package3d_urn="urn:adsk.eagle:package:23507/1" value="4.7uH" x="4.25" y="19">
+<attribute name="SPICEPREFIX" value="L" x="4.25" y="19" size="1.778" layer="27" display="off"/>
+</element>
 <element name="U11" library="MCP1642B" package="MCP1642B" value="MCP1642B" x="11.5" y="20" rot="R180"/>
 </elements>
