File: TPS61032.brd (EAGLE design)
At the start: 21.6 x 49.2 mm, 11 parts, among them U1 TPS61032PWPRPWP16_2P31X2P46-L

Commit message: Fri 17 May 2019 16:01:28 EDT - added README.md
Changed lines of the file:
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@@
 <?xml version="1.0" encoding="utf-8"?>
 <!DOCTYPE eagle SYSTEM "eagle.dtd">
-<eagle version="9.0.0">
+<eagle version="9.4.0">
 <drawing>
 <settings>
-<setting alwaysvectorfont="no"/>
+<setting alwaysvectorfont="yes"/>
 <setting verticaltext="up"/>
 </settings>
@@
 <param name="checkStop" value="0"/>
 <param name="checkValues" value="0"/>
+<param name="checkNames" value="1"/>
+<param name="checkWireStubs" value="1"/>
+<param name="checkPolygonWidth" value="0"/>
 <param name="useDiameter" value="13"/>
 <param name="maxErrors" value="50"/>
@@
 </autorouter>
 <elements>
-<element name="C1" library="Seeed-Capacitor" library_urn="urn:adsk.eagle:library:464" package="C0805" package3d_urn="urn:adsk.eagle:package:32459/1" value="10uf/6V/X7R" x="20.32" y="20.32" rot="R180">
+<element name="C1" library="Seeed-Capacitor" library_urn="urn:adsk.eagle:library:464" package="C0805" package3d_urn="urn:adsk.eagle:package:32459/1" value="10uf/6V/X7R" x="20.32" y="20.32" smashed="yes" rot="R180">
 <attribute name="MPN" value="CC0805ZKY5V6BB106" x="20.32" y="20.32" size="1.778" layer="27" rot="R180" display="off"/>
-</element>
-<element name="C2" library="Seeed-Capacitor" library_urn="urn:adsk.eagle:library:464" package="C0805" package3d_urn="urn:adsk.eagle:package:32459/1" value="10uf/6V/X7R" x="5.08" y="36.83" rot="R180">
+<attribute name="NAME" x="19.177" y="18.415" size="0.889" layer="25" font="vector" ratio="11" rot="R90"/>
+<attribute name="VALUE" x="22.479" y="18.415" size="0.635" layer="27" ratio="10" rot="R90"/>
+</element>
+<element name="C2" library="Seeed-Capacitor" library_urn="urn:adsk.eagle:library:464" package="C0805" package3d_urn="urn:adsk.eagle:package:32459/1" value="10uf/6V/X7R" x="5.08" y="36.83" smashed="yes" rot="R180">
 <attribute name="MPN" value="CC0805ZKY5V6BB106" x="5.08" y="36.83" size="1.778" layer="27" rot="R180" display="off"/>
-</element>
-<element name="C3" library="Seeed-Capacitor" library_urn="urn:adsk.eagle:library:464" package="AVX-D" package3d_urn="urn:adsk.eagle:package:32385/1" value="470uf" x="16.51" y="35.56" rot="R270">
+<attribute name="NAME" x="3.937" y="34.925" size="0.889" layer="25" font="vector" ratio="11" rot="R90"/>
+<attribute name="VALUE" x="7.239" y="34.925" size="0.635" layer="27" ratio="10" rot="R90"/>
+</element>
+<element name="C3" library="Seeed-Capacitor" library_urn="urn:adsk.eagle:library:464" package="AVX-D" package3d_urn="urn:adsk.eagle:package:32385/1" value="470uf" x="16.51" y="35.56" smashed="yes" rot="R270">
 <attribute name="MPN" value="TAJD477*006#NJ" x="16.51" y="35.56" size="1.778" layer="27" rot="R270" display="off"/>
-</element>
-<element name="D1" library="Seeed-LED" library_urn="urn:adsk.eagle:library:472" package="LED-0603" package3d_urn="urn:adsk.eagle:package:32743/1" value="BLUE-0603" x="11.43" y="39.37" rot="R180">
+<attribute name="NAME" x="19.05" y="39.37" size="0.889" layer="25" ratio="11" rot="R270"/>
+<attribute name="VALUE" x="13.208" y="39.37" size="0.635" layer="27" ratio="10" rot="R270"/>
+</element>
+<element name="D1" library="Seeed-LED" library_urn="urn:adsk.eagle:library:472" package="LED-0603" package3d_urn="urn:adsk.eagle:package:32743/1" value="BLUE-0603" x="11.43" y="39.37" smashed="yes" rot="R180">
 <attribute name="MPN" value="19-217-BHC-ZL1M2RY-3T" x="11.43" y="39.37" size="1.778" layer="27" rot="R180" display="off"/>
-</element>
-<element name="J1" library="SparkFun-Connectors" library_urn="urn:adsk.eagle:library:513" package="JST-2-SMD" package3d_urn="urn:adsk.eagle:package:38042/1" value="" x="10.16" y="5.08" rot="R180">
+<attribute name="NAME" x="13.335" y="38.481" size="0.889" layer="25" ratio="11" rot="R180"/>
+<attribute name="VALUE" x="12.573" y="40.9575" size="0.635" layer="27" ratio="10" rot="R180"/>
+</element>
+<element name="J1" library="SparkFun-Connectors" library_urn="urn:adsk.eagle:library:513" package="JST-2-SMD" package3d_urn="urn:adsk.eagle:package:38042/1" value="" x="10.16" y="5.08" smashed="yes" rot="R180">
+<attribute name="NAME" x="11.557" y="3.302" size="0.6096" layer="25" font="vector" ratio="20" rot="R180"/>
 <attribute name="PROD_ID" value="CONN-11443" x="10.16" y="5.08" size="1.778" layer="27" rot="R180" display="off"/>
 <attribute name="SF_ID" value="PRT-08612" x="10.16" y="5.08" size="1.778" layer="27" rot="R180" display="off"/>
-</element>
-<element name="J2" library="SparkFun-Connectors" library_urn="urn:adsk.eagle:library:513" package="1X02_XTRA_BIG" package3d_urn="urn:adsk.eagle:package:38054/1" value="" x="12.7" y="45.72" rot="R180"/>
-<element name="L1" library="mw-wurth" package="7443550820" value="8.2uH" x="10.16" y="20.32" rot="R180"/>
-<element name="R1" library="Seeed-Resistor" library_urn="urn:adsk.eagle:library:474" package="R0805" package3d_urn="urn:adsk.eagle:package:32799/1" value="269K/1%" x="20.32" y="25.4">
+<attribute name="VALUE" x="11.811" y="4.445" size="0.6096" layer="27" font="vector" ratio="20" rot="R180"/>
+</element>
+<element name="J2" library="SparkFun-Connectors" library_urn="urn:adsk.eagle:library:513" package="1X02_XTRA_BIG" package3d_urn="urn:adsk.eagle:package:38054/1" value="" x="12.7" y="45.72" smashed="yes" rot="R180">
+<attribute name="NAME" x="17.78" y="43.053" size="0.6096" layer="25" font="vector" ratio="20" rot="R180"/>
+<attribute name="VALUE" x="17.78" y="49.022" size="0.6096" layer="27" font="vector" ratio="20" rot="R180"/>
+</element>
+<element name="L1" library="mw-wurth" package="7443550820" value="8.2uH" x="10.16" y="20.32" smashed="yes" rot="R180">
+<attribute name="NAME" x="16.51" y="12.7" size="1.27" layer="21" font="vector" ratio="14" rot="R180"/>
+</element>
+<element name="R1" library="Seeed-Resistor" library_urn="urn:adsk.eagle:library:474" package="R0805" package3d_urn="urn:adsk.eagle:package:32799/1" value="269K/1%" x="20.32" y="25.4" smashed="yes">
 <attribute name="MPN" value="RC0805JR-07220RL" x="20.32" y="25.4" size="1.778" layer="27" display="off"/>
-</element>
-<element name="R2" library="Seeed-Resistor" library_urn="urn:adsk.eagle:library:474" package="R0805" package3d_urn="urn:adsk.eagle:package:32799/1" value="100K/1%" x="20.32" y="29.21">
+<attribute name="NAME" x="21.336" y="27.305" size="0.889" layer="25" font="vector" ratio="11" rot="R270"/>
+<attribute name="VALUE" x="18.415" y="27.305" size="0.889" layer="27" ratio="11" rot="R270"/>
+</element>
+<element name="R2" library="Seeed-Resistor" library_urn="urn:adsk.eagle:library:474" package="R0805" package3d_urn="urn:adsk.eagle:package:32799/1" value="100K/1%" x="20.32" y="29.21" smashed="yes">
 <attribute name="MPN" value="RC0805JR-07220RL" x="20.32" y="29.21" size="1.778" layer="27" display="off"/>
-</element>
-<element name="R3" library="Seeed-Resistor" library_urn="urn:adsk.eagle:library:474" package="R0603" package3d_urn="urn:adsk.eagle:package:32791/1" value="1K" x="7.62" y="39.37" rot="R270">
+<attribute name="NAME" x="21.336" y="31.115" size="0.889" layer="25" font="vector" ratio="11" rot="R270"/>
+<attribute name="VALUE" x="18.415" y="31.115" size="0.889" layer="27" ratio="11" rot="R270"/>
+</element>
+<element name="R3" library="Seeed-Resistor" library_urn="urn:adsk.eagle:library:474" package="R0603" package3d_urn="urn:adsk.eagle:package:32791/1" value="1K" x="7.62" y="39.37" smashed="yes" rot="R270">
 <attribute name="MPN" value="RC0603FR-071KL" x="7.62" y="39.37" size="1.778" layer="27" rot="R270" display="off"/>
-</element>
-<element name="U1" library="32teeth - TPS61030-32" package="PWP16_2P31X2P46-L" value="TPS61032PWPRPWP16_2P31X2P46-L" x="10.16" y="33.02" rot="R90">
+<attribute name="NAME" x="5.715" y="40.386" size="0.889" layer="25" ratio="11"/>
+<attribute name="VALUE" x="6.015" y="37.935" size="0.635" layer="27" ratio="10"/>
+</element>
+<element name="U1" library="32teeth - TPS61030-32" package="PWP16_2P31X2P46-L" value="TPS61032PWPRPWP16_2P31X2P46-L" x="10.16" y="33.02" smashed="yes" rot="R90">
 <attribute name="MANUFACTURER_PART_NUMBER" value="TPS61032PWPR" x="10.16" y="33.02" size="1.778" layer="27" rot="R90" display="off"/>
+<attribute name="NAME" x="10.795" y="29.7434" size="1.27" layer="25" ratio="6" rot="SR90"/>
 <attribute name="VENDOR" value="Texas Instruments" x="10.16" y="33.02" size="1.778" layer="27" rot="R90" display="off"/>
 </element>
@@
 </signal>
 </signals>
+<mfgpreviewcolors>
+<mfgpreviewcolor name="soldermaskcolor" color="0xC8008000"/>
+<mfgpreviewcolor name="silkscreencolor" color="0xFFFEFEFE"/>
+<mfgpreviewcolor name="backgroundcolor" color="0xFF282828"/>
+<mfgpreviewcolor name="coppercolor" color="0xFFFFBF00"/>
+<mfgpreviewcolor name="substratecolor" color="0xFF786E46"/>
+</mfgpreviewcolors>
 </board>
 </drawing>
