File: TPS61099x.brd (EAGLE design)
At the start: 35 x 12 mm, 9 parts, among them J3 Batt Conn

Commit message: Fri 17 May 2019 16:01:28 EDT - added README.md
Changed lines of the file:
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@@
 <?xml version="1.0" encoding="utf-8"?>
 <!DOCTYPE eagle SYSTEM "eagle.dtd">
-<eagle version="9.0.0">
+<eagle version="9.4.0">
 <drawing>
 <settings>
-<setting alwaysvectorfont="no"/>
+<setting alwaysvectorfont="yes"/>
 <setting verticaltext="up"/>
 </settings>
@@
 <param name="checkStop" value="0"/>
 <param name="checkValues" value="0"/>
+<param name="checkNames" value="1"/>
+<param name="checkWireStubs" value="1"/>
+<param name="checkPolygonWidth" value="0"/>
 <param name="useDiameter" value="13"/>
 <param name="maxErrors" value="50"/>
@@
 </autorouter>
 <elements>
-<element name="U$1" library="32teeth - TPS61099x" package="TPS61099X" value="TPS61099X" x="16" y="6.5"/>
-<element name="J3" library="SparkFun-Connectors" package="JST-2-SMD" value="Batt Conn" x="31" y="6" rot="R270">
+<element name="U$1" library="32teeth - TPS61099x" package="TPS61099X" value="TPS61099X" x="16" y="6.5" smashed="yes">
+<attribute name="NAME" x="13.46" y="6.5" size="1.27" layer="25" rot="R90" align="center"/>
+<attribute name="VALUE" x="18.54" y="6.5" size="1.27" layer="27" rot="R270" align="center"/>
+</element>
+<element name="J3" library="SparkFun-Connectors" package="JST-2-SMD" value="Batt Conn" x="31" y="6" smashed="yes" rot="R270">
 <attribute name="BTM_NEG" value="-" x="83.07" y="16.16" size="1.778" layer="27" rot="R270" display="off"/>
 <attribute name="BTM_POS" value="+" x="83.07" y="16.16" size="1.778" layer="27" rot="R270" display="off"/>
+<attribute name="NAME" x="32.27" y="7.27" size="0.4064" layer="25" rot="R270"/>
 <attribute name="PROD_ID" value="CONN-11443" x="83.07" y="16.16" size="1.778" layer="27" rot="R270" display="off"/>
 <attribute name="TOP_NEG" value="-" x="83.07" y="16.16" size="1.778" layer="27" rot="R270" display="off"/>
 <attribute name="TOP_POS" value="+" x="83.07" y="16.16" size="1.778" layer="27" rot="R270" display="off"/>
-</element>
-<element name="J1" library="SparkFun-Connectors" library_urn="urn:adsk.eagle:library:513" package="1X02_XTRA_BIG" package3d_urn="urn:adsk.eagle:package:38054/1" value="" x="3.5" y="6" rot="R270"/>
-<element name="C1" library="Seeed-Capacitor" library_urn="urn:adsk.eagle:library:464" package="C0805" package3d_urn="urn:adsk.eagle:package:32459/1" value="10uf" x="18" y="10" rot="R270">
+<attribute name="VALUE" x="31" y="7.27" size="0.4064" layer="27" rot="R270"/>
+</element>
+<element name="J1" library="SparkFun-Connectors" library_urn="urn:adsk.eagle:library:513" package="1X02_XTRA_BIG" package3d_urn="urn:adsk.eagle:package:38054/1" value="" x="3.5" y="6" smashed="yes" rot="R270">
+<attribute name="NAME" x="6.167" y="11.08" size="0.6096" layer="25" font="vector" ratio="20" rot="R270"/>
+<attribute name="VALUE" x="0.198" y="11.08" size="0.6096" layer="27" font="vector" ratio="20" rot="R270"/>
+</element>
+<element name="C1" library="Seeed-Capacitor" library_urn="urn:adsk.eagle:library:464" package="C0805" package3d_urn="urn:adsk.eagle:package:32459/1" value="10uf" x="18" y="10" smashed="yes" rot="R270">
 <attribute name="MPN" value="CC0805MKX5R5BB226" x="9.11" y="64.61" size="1.778" layer="27" rot="R270" display="off"/>
-</element>
-<element name="R1" library="Seeed-Resistor" library_urn="urn:adsk.eagle:library:474" package="R0805" package3d_urn="urn:adsk.eagle:package:32799/1" value="1-MΩ" x="9" y="3" rot="R90">
+<attribute name="NAME" x="19.905" y="8.857" size="0.889" layer="25" font="vector" ratio="11" rot="R180"/>
+<attribute name="VALUE" x="19.905" y="12.159" size="0.635" layer="27" ratio="10" rot="R180"/>
+</element>
+<element name="R1" library="Seeed-Resistor" library_urn="urn:adsk.eagle:library:474" package="R0805" package3d_urn="urn:adsk.eagle:package:32799/1" value="1-MΩ" x="9" y="3" smashed="yes" rot="R90">
 <attribute name="MPN" value="RL0805JR-070R1L" x="15.35" y="-52.88" size="1.778" layer="27" rot="R90" display="off"/>
-</element>
-<element name="C2" library="Seeed-Capacitor" library_urn="urn:adsk.eagle:library:464" package="C0805" package3d_urn="urn:adsk.eagle:package:32459/1" value="10uf" x="11" y="8" rot="R180">
+<attribute name="NAME" x="7.095" y="4.016" size="0.889" layer="25" font="vector" ratio="11"/>
+<attribute name="VALUE" x="7.095" y="1.095" size="0.889" layer="27" ratio="11"/>
+</element>
+<element name="C2" library="Seeed-Capacitor" library_urn="urn:adsk.eagle:library:464" package="C0805" package3d_urn="urn:adsk.eagle:package:32459/1" value="10uf" x="11" y="8" smashed="yes" rot="R180">
 <attribute name="MPN" value="CC0805MKX5R5BB226" x="11" y="8" size="1.778" layer="27" rot="R180" display="off"/>
-</element>
-<element name="C3" library="Seeed-Capacitor" library_urn="urn:adsk.eagle:library:464" package="C0805" package3d_urn="urn:adsk.eagle:package:32459/1" value="10uf" x="8" y="8" rot="R180">
+<attribute name="NAME" x="9.857" y="6.095" size="0.889" layer="25" font="vector" ratio="11" rot="R90"/>
+<attribute name="VALUE" x="13.159" y="6.095" size="0.635" layer="27" ratio="10" rot="R90"/>
+</element>
+<element name="C3" library="Seeed-Capacitor" library_urn="urn:adsk.eagle:library:464" package="C0805" package3d_urn="urn:adsk.eagle:package:32459/1" value="10uf" x="8" y="8" smashed="yes" rot="R180">
 <attribute name="MPN" value="CC0805MKX5R5BB226" x="8" y="8" size="1.778" layer="27" rot="R180" display="off"/>
-</element>
-<element name="R2" library="Seeed-Resistor" library_urn="urn:adsk.eagle:library:474" package="R0805" package3d_urn="urn:adsk.eagle:package:32799/1" value="249-kΩ" x="14" y="3" rot="R90">
+<attribute name="NAME" x="6.857" y="6.095" size="0.889" layer="25" font="vector" ratio="11" rot="R90"/>
+<attribute name="VALUE" x="10.159" y="6.095" size="0.635" layer="27" ratio="10" rot="R90"/>
+</element>
+<element name="R2" library="Seeed-Resistor" library_urn="urn:adsk.eagle:library:474" package="R0805" package3d_urn="urn:adsk.eagle:package:32799/1" value="249-kΩ" x="14" y="3" smashed="yes" rot="R90">
 <attribute name="MPN" value="RL0805JR-070R1L" x="14" y="3" size="1.778" layer="27" rot="R90" display="off"/>
-</element>
-<element name="L1" library="PowerMagnetics (rev18e)" package="WE-LQS_2512" value="2.2uH" x="21.5" y="5" rot="R180">
+<attribute name="NAME" x="12.095" y="4.016" size="0.889" layer="25" font="vector" ratio="11"/>
+<attribute name="VALUE" x="12.095" y="1.095" size="0.889" layer="27" ratio="11"/>
+</element>
+<element name="L1" library="PowerMagnetics (rev18e)" package="WE-LQS_2512" value="2.2uH" x="21.5" y="5" smashed="yes" rot="R180">
+<attribute name="NAME" x="21.44" y="3.06" size="0.6096" layer="25" rot="R180" align="bottom-center"/>
+<attribute name="VALUE" x="22.84" y="7.31" size="0.6096" layer="27" rot="R180"/>
 <attribute name="WE-NUMBER" value="74404024022/2,2uH" x="21.5" y="5" size="1.778" layer="27" rot="R180" display="off"/>
 </element>
@@
 <contactref element="R2" pad="2"/>
 <contactref element="U$1" pad="GND"/>
-<polygon width="0.1524" layer="1">
+<polygon width="0.1524" layer="1" thermals="no">
 <vertex x="0" y="12"/>
 <vertex x="35" y="12"/>
@@
 <vertex x="0" y="0"/>
 </polygon>
-<polygon width="0.1524" layer="16">
+<polygon width="0.1524" layer="16" thermals="no">
 <vertex x="0" y="12"/>
 <vertex x="35" y="12"/>
@@
 </signal>
 </signals>
+<mfgpreviewcolors>
+<mfgpreviewcolor name="soldermaskcolor" color="0xC8008000"/>
+<mfgpreviewcolor name="silkscreencolor" color="0xFFFEFEFE"/>
+<mfgpreviewcolor name="backgroundcolor" color="0xFF282828"/>
+<mfgpreviewcolor name="coppercolor" color="0xFFFFBF00"/>
+<mfgpreviewcolor name="substratecolor" color="0xFF786E46"/>
+</mfgpreviewcolors>
 <errors>
 </errors>
